Commit message: Add files via upload

File: Robot Assembly.SLDASM/urdf/Robot Assembly.SLDASM.urdf (robot description, URDF)
Before this commit: robot Robot Assembly.SLDASM, 7 links, 6 joints
Links:
- removed link Link2_R
- removed link Link3_Elb
- removed link Link4_Wr
- removed link Link5_EE
- added link Link3_R, mass 5.5098; collision mesh filename=package://Robot Assembly.SLDASM/meshes/Link3_R.STL; visual mesh filename=package://Robot Assembly.SLDASM/meshes/Link3_R.STL
- added link Link4, mass 0.10865; collision mesh filename=package://Robot Assembly.SLDASM/meshes/Link4.STL; visual mesh filename=package://Robot Assembly.SLDASM/meshes/Link4.STL
- added link Link5, mass 0.052656; collision mesh filename=package://Robot Assembly.SLDASM/meshes/Link5.STL; visual mesh filename=package://Robot Assembly.SLDASM/meshes/Link5.STL
- added link Link6, mass 0.05213; collision mesh filename=package://Robot Assembly.SLDASM/meshes/Link6.STL; visual mesh filename=package://Robot Assembly.SLDASM/meshes/Link6.STL
- added link Pen_tip, mass 5.5098; collision mesh filename=package://Robot Assembly.SLDASM/meshes/Pen_tip.STL; visual mesh filename=package://Robot Assembly.SLDASM/meshes/Pen_tip.STL
- link Link1: mass 0.251146740283358 -> 0.25963
- link Link2_L: mass 0.114015670147046 -> 0.11526
- link base_link: mass 0.866068274339261 -> 0.70117
Joints:
- removed joint Link1
- removed joint Link2_L
- removed joint Link2_R
- removed joint Link3_Elb
- removed joint Link4_Wr
- removed joint Link5_EE
- added joint Joint_EE: type revolute, parent Link5, child Link6, origin xyz=0.021626 -0.020046 -0.00367 rpy=0 0 0, axis 0.98598 0.01164 -0.16646, limit lower=-0.6981 upper=2.0944 effort=1.5 velocity=6.18
- added joint Motor1_joint: type revolute, parent base_link, child Link1, origin xyz=0 0 0.0507 rpy=0 0 0, axis 0 0 1, limit lower=-1.0472 upper=0.6981 effort=1.5 velocity=6.18
- added joint Motor2_L: type revolute, parent Link1, child Link2_L, origin xyz=0.052457 0.00059405 0.0483 rpy=0 0 0, axis 0.99994 0.011324 0, limit lower=0 upper=6.283 effort=6 velocity=6.6
- added joint Motor3_R: type revolute, parent Link1, child Link3_R, origin xyz=-0.052457 -0.00059406 0.0483 rpy=0 0 0, axis -0.99994 -0.011324 0, limit lower=-1.0472 upper=1.0472 effort=6 velocity=6.6, mimic joint=Motor2_L multiplier=-1 offset=0
- added joint Motor4_elb: type revolute, parent Link2_L, child Link4, origin xyz=-0.072748 -0.12514 0.1444 rpy=0 0 0, axis -0.99994 -0.011324 0, limit lower=-2.4435 upper=1.0472 effort=1.5 velocity=6.18
- added joint Motor5_wr: type revolute, parent Link4, child Link5, origin xyz=0.02195 -0.021925 0.17994 rpy=0 0 0, axis 0.011324 -0.99993 -0.0028474, limit lower=-1.3963 upper=1.3963 effort=1.5 velocity=6.18
- added joint Pen_tip: type fixed, parent Link6, child Pen_tip, origin xyz=-0.021396 -0.18979 -0.0096416 rpy=0 0 0, axis 0 0 0
