Commit message: Align online/offline ACE planning and update simple_robot_v2 assets

File: online/src/me557_pen_description/urdf/Robot Assembly.SLDASM.urdf (robot description, URDF)
Before this commit: robot Robot Assembly.SLDASM, 9 links, 8 joints
Links:
- link Link1: mass 0.25963 -> 0.24905
- link Link2_L: mass 0.11526 -> 0.12701
- link Link4: mass 0.10865 -> 0.083206
- link Link5: mass 0.052656 -> 0.053757
- link Link6: mass 0.05213 -> 0.081357
- link Pen_tip: mass 5.5098 -> 0.00038082; geometry collision mesh filename=package://me557_pen_description/meshes/Pen_tip.STL; visual mesh filename=package://me557_pen_description/meshes/Pen_tip.STL
- link base_link: mass 0.70117 -> 0.49574
Joints:
- removed joint Pen_tip
- added joint pen_tip_fixed: type fixed, parent Link6, child Pen_tip, origin xyz=0.17403 0.0375 -0.00098 rpy=1.5708 -1.5643 1.5708
- joint Joint_EE: axis 0.98598 0.01164 -0.16646 -> 0 0 1; limit lower=-0.6981 upper=2.0944 effort=1.5 velocity=6.18 -> lower=-1.1781 upper=1.1781 effort=0 velocity=0; origin xyz=0.021626 -0.020046 -0.00367 rpy=0 0 0 -> xyz=0 -0.001 0.041 rpy=1.5708 0 0
- joint Motor1_joint: axis 0 0 1 -> 0 0 -1; limit lower=-1.0472 upper=0.6981 effort=1.5 velocity=6.18 -> lower=-0.87265 upper=0.87265 effort=0 velocity=0; origin xyz=0 0 0.0507 rpy=0 0 0 -> xyz=0 0 0.05 rpy=0 0 0
- joint Motor2_L: axis 0.99994 0.011324 0 -> 0 0 1; limit lower=0 upper=6.283 effort=6 velocity=6.6 -> lower=-1.047195 upper=1.047195 effort=0 velocity=0; origin xyz=0.052457 0.00059405 0.0483 rpy=0 0 0 -> xyz=0 0 0.049 rpy=1.5708 0 0.0064475
- joint Motor4_elb: axis -0.99994 -0.011324 0 -> 0 0 1; limit lower=-2.4435 upper=1.0472 effort=1.5 velocity=6.18 -> lower=-1.876225 upper=1.876225 effort=0 velocity=0; origin xyz=-0.072748 -0.12514 0.1444 rpy=0 0 0 -> xyz=0 0.2247 0.00104 rpy=0 0 0
- joint Motor5_wr: axis 0.011324 -0.99993 -0.0028474 -> 0 0 -1; limit lower=-1.3963 upper=1.3963 effort=1.5 velocity=6.18 -> lower=-0.95995 upper=0.95995 effort=0 velocity=0; origin xyz=0.02195 -0.021925 0.17994 rpy=0 0 0 -> xyz=0.00108 0.0935 -0.001 rpy=1.5708 0 1.5708
- joint base_to_floor: origin xyz=0 -0.91 -0.01 rpy=0 0 0 -> xyz=0.91 0 -0.01 rpy=0 0 1.5708

File: online/src/me557_pen_description/urdf/me557_pen.urdf (robot description, URDF)
Before this commit: robot me557_pen, 9 links, 8 joints
Links:
- link Link1: mass 0.25963 -> 0.24905
- link Link2_L: mass 0.11526 -> 0.12701
- link Link4: mass 0.10865 -> 0.083206
- link Link5: mass 0.052656 -> 0.053757
- link Link6: mass 0.05213 -> 0.081357
- link Pen_tip: mass 5.5098 -> 0.00038082; geometry collision mesh filename=package://me557_pen_description/meshes/Pen_tip.STL; visual mesh filename=package://me557_pen_description/meshes/Pen_tip.STL
- link base_link: mass 0.70117 -> 0.49574
Joints:
- joint Joint_EE: axis 0.98598 0.01164 -0.16646 -> 0 0 1; limit lower=-0.6981 upper=2.0944 effort=1.5 velocity=6.18 -> lower=-1.1781 upper=1.1781 effort=0 velocity=0; origin xyz=0.021626 -0.020046 -0.00367 rpy=0 0 0 -> xyz=0 -0.001 0.041 rpy=1.5708 0 0
- joint Motor1_joint: axis 0 0 1 -> 0 0 -1; limit lower=-1.0472 upper=0.6981 effort=1.5 velocity=6.18 -> lower=-0.87265 upper=0.87265 effort=0 velocity=0; origin xyz=0 0 0.0507 rpy=0 0 0 -> xyz=0 0 0.05 rpy=0 0 0
- joint Motor2_L: axis 0.99994 0.011324 0 -> 0 0 1; limit lower=0 upper=6.283 effort=6 velocity=6.6 -> lower=-1.047195 upper=1.047195 effort=0 velocity=0; origin xyz=0.052457 0.00059405 0.0483 rpy=0 0 0 -> xyz=0 0 0.049 rpy=1.5708 0 0.0064475
- joint Motor4_elb: axis -0.99994 -0.011324 0 -> 0 0 1; limit lower=-2.4435 upper=1.0472 effort=1.5 velocity=6.18 -> lower=-1.876225 upper=1.876225 effort=0 velocity=0; origin xyz=-0.072748 -0.12514 0.1444 rpy=0 0 0 -> xyz=0 0.2247 0.00104 rpy=0 0 0
- joint Motor5_wr: axis 0.011324 -0.99993 -0.0028474 -> 0 0 -1; limit lower=-1.3963 upper=1.3963 effort=1.5 velocity=6.18 -> lower=-0.95995 upper=0.95995 effort=0 velocity=0; origin xyz=0.02195 -0.021925 0.17994 rpy=0 0 0 -> xyz=0.00108 0.0935 -0.001 rpy=1.5708 0 1.5708
- joint base_to_floor: origin xyz=0 -0.91 -0.01 rpy=0 0 0 -> xyz=0.91 0 -0.01 rpy=0 0 1.5708
- joint pen_tip_fixed: axis 0 0 0 -> (none); origin xyz=-0.021396 -0.18979 -0.0096416 rpy=0 0 0 -> xyz=0.17403 0.0375 -0.00098 rpy=1.5708 -1.5643 1.5708
